File: citysensor/hardware/eagle/citysensor.brd (EAGLE design)
At the start: 65.7 x 31.7 mm, 15 parts, among them U1 ATMEGA328P_TQFP, X1 16MHZ

Commit message: add the city sensor parts library
Parts:
- U$1: device fdorothy:PIZERO -> citysensor:PIZERO
- U$2: device fdorothy:TC2030-CLIP -> citysensor:TC2030-CLIP
- X1: device fdorothy:CRYSTAL-M445 -> citysensor:CRYSTAL-M445
Changed lines of the file:
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@@
 <attribute name="NAME" x="23.622" y="19.304" size="1.27" layer="25" rot="R270"/>
 </element>
-<element name="U$1" library="fdorothy" package="PIZERO" value="PIZERO" x="33.02" y="26.67"/>
+<element name="U$1" library="citysensor" package="PIZERO" value="PIZERO" x="33.02" y="26.67"/>
 <element name="U1" library="SparkFun-IC-Microcontroller" library_urn="urn:adsk.eagle:library:525" package="TQFP32-08" package3d_urn="urn:adsk.eagle:package:38945/1" value="ATMEGA328P_TQFP" x="21.59" y="10.16" smashed="yes">
 <attribute name="NAME" x="21.59" y="15.875" size="0.6096" layer="25" font="vector" ratio="20" align="bottom-center"/>
@@
 <attribute name="VALUE" x="22.352" y="4.064" size="0.6096" layer="27" font="vector" ratio="20" align="bottom-center"/>
 </element>
-<element name="X1" library="fdorothy" package="CRYSTAL-M445" value="16MHZ" x="13.97" y="5.08" rot="R90"/>
-<element name="U$2" library="fdorothy" package="TC2030-CLIP" value="TC2030-CLIP" x="4.826" y="13.97" rot="R270"/>
+<element name="X1" library="citysensor" package="CRYSTAL-M445" value="16MHZ" x="13.97" y="5.08" rot="R90"/>
+<element name="U$2" library="citysensor" package="TC2030-CLIP" value="TC2030-CLIP" x="4.826" y="13.97" rot="R270"/>
 </elements>
 <signals>

Commit message: initial board layout for rev2
Parts:
- added C10: 220uF, resistor:153CLV-0505
- added C7, C8, C9: .1uF, resistor:C0805
- added DUST: GP2Y1010AU0F, citysensor:S6B-ZR-SM4A-TF
- added I2C: CON-I2C, citysensor:MOLEX_6
- added MIC: MIC, citysensor:MOLEX_3
- added R6: 150, resistor:M0805
- added R7: 10k, resistor:M0805
- added TEMP: DHT11, citysensor:MOLEX_3
- moved C1 0.28 mm to (29.2, 8.51)
Connections:
- removed net 3V3_2: U$1.P$17
- removed net N$2: C2.2, U1.4
- removed net N$3: C3.2, U1.6
- removed net N$4: C1.2, U1.18
- removed net N$7: R4.2, U1.27
- removed net N$8: R5.2, U1.28
- new net 3V3: C9.2, I2C.P$3, U$1.P$17
- new net DSTA: DUST.P$5, U1.23
- new net DSTLED: DUST.P$3, U1.13
- new net I2C_INT: I2C.P$2, U1.1
- new net MIC_AOUT: MIC.P$1, U1.24
- new net SCL: I2C.P$6, R5.2, U1.28
- new net SDA: I2C.P$5, R4.2, U1.27
- new net THDATA: R7.2, TEMP.P$2, U1.11
- new net V-LED: C10.+, DUST.P$1, R6.1
- net GND: now also C10.-, C7.2, C8.1, C9.1, DUST.P$2, DUST.P$4, I2C.P$4, MIC.P$2, TEMP.P$3, U1.21, U1.3, U1.5
- net VCC: now also C1.2, C2.2, C3.2, C7.1, C8.2, DUST.P$6, I2C.P$1, MIC.P$3, R6.2, R7.1, TEMP.P$1, U1.18, U1.4, U1.6
Routing:
- net VCC: track 39.7 -> 165.9 mm, vias 0 -> 2
- net THDATA: track 0.00 -> 40.4 mm
- net SCL: track 0.00 -> 32.8 mm, vias 0 -> 2
- net MIC_AOUT: track 0.00 -> 31.8 mm
- net SDA: track 0.00 -> 28.9 mm
- net I2C_INT: track 0.00 -> 23.3 mm, vias 0 -> 1
- net 3V3: track 0.00 -> 20.8 mm, vias 0 -> 1
- net DSTLED: track 0.00 -> 20.1 mm
- net DSTA: track 0.00 -> 20.0 mm, vias 0 -> 2
- net N$7: track 7.79 -> 0.00 mm
- net V-LED: track 0.00 -> 7.42 mm
- net N$8: track 7.07 -> 0.00 mm
- net N$2: track 3.61 -> 0.00 mm
- net N$3: track 3.07 -> 0.00 mm
- net N$4: track 2.54 -> 0.00 mm
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