File: citysensor/hardware/eagle/citysensor.sch (EAGLE design)
At the start: 15 parts, among them U1 ATMEGA328P_TQFP, X1 16MHZ

Commit message: add the city sensor parts library
Parts:
- U$1: device fdorothy:PIZERO -> citysensor:PIZERO
- U$2: device fdorothy:TC2030-CLIP -> citysensor:TC2030-CLIP
- X1: device fdorothy:CRYSTAL-M445 -> citysensor:CRYSTAL-M445
Changed lines of the file:
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@@
 </classes>
 <parts>
-<part name="U$1" library="fdorothy" deviceset="PIZERO" device=""/>
+<part name="U$1" library="citysensor" deviceset="PIZERO" device=""/>
 <part name="U1" library="SparkFun-IC-Microcontroller" library_urn="urn:adsk.eagle:library:525" deviceset="ATMEGA328P_TQFP" device="" package3d_urn="urn:adsk.eagle:package:38945/1" value="ATMEGA328P_TQFP"/>
 <part name="GND1" library="supply1" library_urn="urn:adsk.eagle:library:371" deviceset="GND" device=""/>
@@
 <part name="C3" library="resistor" library_urn="urn:adsk.eagle:library:348" deviceset="C-EU" device="C0805" package3d_urn="urn:adsk.eagle:package:26137/1" value=".1uF"/>
 <part name="GND2" library="supply1" library_urn="urn:adsk.eagle:library:371" deviceset="GND" device=""/>
-<part name="X1" library="fdorothy" deviceset="CRYSTAL-M445" device="" value="16MHZ"/>
+<part name="X1" library="citysensor" deviceset="CRYSTAL-M445" device="" value="16MHZ"/>
 <part name="C4" library="resistor" library_urn="urn:adsk.eagle:library:348" deviceset="C-EU" device="C0805" package3d_urn="urn:adsk.eagle:package:26137/1" value="22pF"/>
 <part name="C5" library="resistor" library_urn="urn:adsk.eagle:library:348" deviceset="C-EU" device="C0805" package3d_urn="urn:adsk.eagle:package:26137/1" value="22pF"/>
@@
 <part name="R4" library="resistor" library_urn="urn:adsk.eagle:library:348" deviceset="R-EU_" device="M0805" package3d_urn="urn:adsk.eagle:package:26079/1" value="4k7"/>
 <part name="R5" library="resistor" library_urn="urn:adsk.eagle:library:348" deviceset="R-EU_" device="M0805" package3d_urn="urn:adsk.eagle:package:26079/1" value="4k7"/>
-<part name="U$2" library="fdorothy" deviceset="TC2030-CLIP" device=""/>
+<part name="U$2" library="citysensor" deviceset="TC2030-CLIP" device=""/>
 </parts>
 <sheets>

Commit message: initial board layout for rev2
Parts:
- added C10: 220uF, resistor:CPOL-US153CLV-0505
- added C7, C8, C9: .1uF, resistor:C-EUC0805
- added DUST: GP2Y1010AU0F, citysensor:GP2Y1010AU0F
- added I2C: CON-I2C, citysensor:CON-I2C
- added MIC: MIC, citysensor:MIC
- added R6: 150, resistor:R-EU_M0805
- added R7: 10k, resistor:R-EU_M0805
- added TEMP: DHT11, citysensor:DHT11
Connections:
- removed net N$2: C2.2, U1.VCC@4
- removed net N$3: C3.2, U1.VCC@6
- removed net N$4: C1.2, U1.AVCC
- removed net N$7: R4.2, U1.PC4(ADC4/SDA)
- removed net N$8: R5.2, U1.PC5(ADC5/SCL)
- new net 3V3: C9.2, I2C.3V3, U$1.3V3_2
- new net DSTA: DUST.VO, U1.PC0(ADC0)
- new net DSTLED: DUST.LED, U1.PB1(OC1A)
- new net I2C_INT: I2C.D3, U1.PD3(INT1)
- new net MIC_AOUT: MIC.AO, U1.PC1(ADC1)
- new net SCL: I2C.SCL, R5.2, U1.PC5(ADC5/SCL)
- new net SDA: I2C.SDA, R4.2, U1.PC4(ADC4/SDA)
- new net THDATA: R7.2, TEMP.DATA, U1.PD7(AIN1)
- new net V-LED: C10.+, DUST.V-LED, R6.1
- net GND: now also C10.-, C7.2, C8.1, C9.1, DUST.LED-GND, DUST.S-GND, I2C.GND, MIC.GND, TEMP.GND, U$1.GND@2, U1.AGND, U1.GND@3, U1.GND@5
- net VCC: now also C1.2, C2.2, C3.2, C7.1, C8.2, DUST.VCC, I2C.VCC, MIC.VCC, R6.2, R7.1, TEMP.VCC, U1.AVCC, U1.VCC@4, U1.VCC@6

Commit message: hooked up reset pin
Connections:
- net PIRESET: now also U$1.GPIO17
Changed lines of the file:
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@@
 <segment>
 <pinref part="U1" gate="U$1" pin="PD0(RXD)"/>
-<wire x1="175.26" y1="48.26" x2="177.8" y2="48.26" width="0.1524" layer="91"/>
-<label x="177.8" y="48.26" size="1.778" layer="95"/>
+<wire x1="175.26" y1="48.26" x2="182.88" y2="48.26" width="0.1524" layer="91"/>
+<label x="182.88" y="48.26" size="1.778" layer="95"/>
 </segment>
 </net>
@@
 <segment>
 <pinref part="U1" gate="U$1" pin="PD1(TXD)"/>
-<wire x1="175.26" y1="45.72" x2="177.8" y2="45.72" width="0.1524" layer="91"/>
-<label x="177.8" y="45.72" size="1.778" layer="95"/>
+<wire x1="175.26" y1="45.72" x2="182.88" y2="45.72" width="0.1524" layer="91"/>
+<label x="182.88" y="45.72" size="1.778" layer="95"/>
 </segment>
 <segment>
@@
 <label x="134.62" y="96.52" size="1.778" layer="95"/>
 </segment>
+<segment>
+<pinref part="U$1" gate="G$1" pin="GPIO17"/>
+<wire x1="15.24" y1="58.42" x2="7.62" y2="58.42" width="0.1524" layer="91"/>
+<label x="2.54" y="58.42" size="1.778" layer="95"/>
+</segment>
 </net>
 <net name="VCC" class="0">
@@
 <segment>
 <pinref part="U1" gate="U$1" pin="PD3(INT1)"/>
-<wire x1="175.26" y1="40.64" x2="177.8" y2="40.64" width="0.1524" layer="91"/>
-<label x="177.8" y="40.64" size="1.778" layer="95"/>
-</segment>
-<segment>
+<wire x1="175.26" y1="40.64" x2="182.88" y2="40.64" width="0.1524" layer="91"/>
+<label x="182.88" y="40.64" size="1.778" layer="95"/>
+</segment>
+<segment>

Commit message: added switch locations to eagle file
Parts:
- added BTN1, BTN2: BTN, citysensor:BTN
- added R8, R9: 10k, resistor:R-EU_M0805
Connections:
- new net BTN1OUT: BTN1.OUT, R8.1, U$1.GPIO13
- new net BTN2OUT: BTN2.OUT, R9.1, U$1.GPIO06
- net GND: now also R8.2, R9.2
- net VCC: now also BTN1.VCC, BTN2.VCC
Changed lines of the file:
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@@
 <part name="GND4" library="supply1" library_urn="urn:adsk.eagle:library:371" deviceset="GND" device=""/>
 <part name="GND5" library="supply1" library_urn="urn:adsk.eagle:library:371" deviceset="GND" device=""/>
+<part name="BTN1" library="citysensor" deviceset="BTN" device=""/>
+<part name="BTN2" library="citysensor" deviceset="BTN" device=""/>
+<part name="R8" library="resistor" library_urn="urn:adsk.eagle:library:348" deviceset="R-EU_" device="M0805" package3d_urn="urn:adsk.eagle:package:26079/1" value="10k"/>
+<part name="R9" library="resistor" library_urn="urn:adsk.eagle:library:348" deviceset="R-EU_" device="M0805" package3d_urn="urn:adsk.eagle:package:26079/1" value="10k"/>
+<part name="GND6" library="supply1" library_urn="urn:adsk.eagle:library:371" deviceset="GND" device=""/>
 </parts>
 <sheets>
@@
 <instance part="GND4" gate="1" x="228.6" y="50.8"/>
 <instance part="GND5" gate="1" x="119.38" y="12.7"/>
+<instance part="BTN1" gate="G$1" x="83.82" y="12.7"/>
+<instance part="BTN2" gate="G$1" x="83.82" y="-7.62"/>
+<instance part="R8" gate="G$1" x="66.04" y="10.16" rot="R180"/>
+<instance part="R9" gate="G$1" x="66.04" y="-10.16" rot="R180"/>
+<instance part="GND6" gate="1" x="55.88" y="-17.78"/>
 </instances>
 <busses>
@@
 <junction x="119.38" y="15.24"/>
 </segment>
+<segment>
+<pinref part="R8" gate="G$1" pin="2"/>
+<pinref part="GND6" gate="1" pin="GND"/>
+<wire x1="60.96" y1="10.16" x2="55.88" y2="10.16" width="0.1524" layer="91"/>
+<wire x1="55.88" y1="10.16" x2="55.88" y2="-10.16" width="0.1524" layer="91"/>
+<pinref part="R9" gate="G$1" pin="2"/>
+<wire x1="55.88" y1="-10.16" x2="55.88" y2="-15.24" width="0.1524" layer="91"/>
+<wire x1="60.96" y1="-10.16" x2="55.88" y2="-10.16" width="0.1524" layer="91"/>
+<junction x="55.88" y="-10.16"/>
+</segment>
 </net>
 <net name="N$5" class="0">
@@
 <label x="121.92" y="66.04" size="1.778" layer="95"/>
 </segment>
+<segment>
+<pinref part="BTN1" gate="G$1" pin="VCC"/>
+<wire x1="78.74" y1="15.24" x2="73.66" y2="15.24" width="0.1524" layer="91"/>
+<label x="71.12" y="15.24" size="1.778" layer="95"/>
+</segment>
+<segment>
+<pinref part="BTN2" gate="G$1" pin="VCC"/>
+<wire x1="78.74" y1="-5.08" x2="73.66" y2="-5.08" width="0.1524" layer="91"/>
+<label x="71.12" y="-5.08" size="1.778" layer="95"/>
+</segment>
 </net>
 <net name="MISO" class="0">
@@
 </segment>
 </net>
+<net name="BTN1OUT" class="0">
+<segment>
+<pinref part="R8" gate="G$1" pin="1"/>
+<pinref part="BTN1" gate="G$1" pin="OUT"/>
+<wire x1="71.12" y1="10.16" x2="78.74" y2="10.16" width="0.1524" layer="91"/>
+<label x="71.374" y="7.366" size="1.778" layer="95"/>
+</segment>
+<segment>
+<pinref part="U$1" gate="G$1" pin="GPIO13"/>
+<wire x1="15.24" y1="30.48" x2="7.62" y2="30.48" width="0.1524" layer="91"/>
+<label x="7.62" y="30.48" size="1.778" layer="95"/>
+</segment>
+</net>
+<net name="BTN2OUT" class="0">
+<segment>
+<pinref part="BTN2" gate="G$1" pin="OUT"/>
+<pinref part="R9" gate="G$1" pin="1"/>
+<wire x1="78.74" y1="-10.16" x2="71.12" y2="-10.16" width="0.1524" layer="91"/>
+<label x="71.374" y="-12.954" size="1.778" layer="95"/>
+</segment>
+<segment>
+<pinref part="U$1" gate="G$1" pin="GPIO06"/>
+<wire x1="15.24" y1="33.02" x2="7.62" y2="33.02" width="0.1524" layer="91"/>
+<label x="7.62" y="33.02" size="1.778" layer="95"/>
+</segment>
+</net>

Commit message: added an rgbled component to the city sensor lib. Added a normal led to the board for arduino status
Parts:
- added LED1: (no value), adafruit:LEDCHIP-LED0805
- added R10, R11: 1k, resistor:R-EU_M0805
- added R12: 330, resistor:R-EU_M0805
Connections:
- new net N$1: BTN1.VCC, R10.2
- new net N$2: BTN2.VCC, R11.2
- new net N$3: R12.1, U1.PD5(T1)
- new net N$4: LED1.C, R12.2
- net GND: now also LED1.A
- net VCC: now also R10.1, R11.1; no longer BTN1.VCC, BTN2.VCC
Other:
- moved on the sheet: BTN1, R8
Changed lines of the file:
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@@
 <layer number="230" name="230bmp" color="7" fill="1" visible="yes" active="yes"/>
 <layer number="231" name="231bmp" color="7" fill="1" visible="yes" active="yes"/>
+<layer number="232" name="Eagle3D_PG2" color="7" fill="1" visible="no" active="no"/>
+<layer number="233" name="Eagle3D_PG3" color="7" fill="1" visible="no" active="no"/>
 <layer number="248" name="Housing" color="7" fill="1" visible="yes" active="yes"/>
 <layer number="249" name="Edge" color="7" fill="1" visible="yes" active="yes"/>
@@
 <part name="R9" library="resistor" library_urn="urn:adsk.eagle:library:348" deviceset="R-EU_" device="M0805" package3d_urn="urn:adsk.eagle:package:26079/1" value="10k"/>
 <part name="GND6" library="supply1" library_urn="urn:adsk.eagle:library:371" deviceset="GND" device=""/>
+<part name="R10" library="resistor" library_urn="urn:adsk.eagle:library:348" deviceset="R-EU_" device="M0805" package3d_urn="urn:adsk.eagle:package:26079/1" value="1k"/>
+<part name="R11" library="resistor" library_urn="urn:adsk.eagle:library:348" deviceset="R-EU_" device="M0805" package3d_urn="urn:adsk.eagle:package:26079/1" value="1k"/>
+<part name="R12" library="resistor" library_urn="urn:adsk.eagle:library:348" deviceset="R-EU_" device="M0805" package3d_urn="urn:adsk.eagle:package:26079/1" value="330"/>
+<part name="LED1" library="adafruit" deviceset="LED" device="CHIP-LED0805"/>
 </parts>
 <sheets>
@@
 <instance part="GND4" gate="1" x="228.6" y="50.8"/>
 <instance part="GND5" gate="1" x="119.38" y="12.7"/>
-<instance part="BTN1" gate="G$1" x="83.82" y="12.7"/>
+<instance part="BTN1" gate="G$1" x="83.82" y="20.32"/>
 <instance part="BTN2" gate="G$1" x="83.82" y="-7.62"/>
-<instance part="R8" gate="G$1" x="66.04" y="10.16" rot="R180"/>
+<instance part="R8" gate="G$1" x="66.04" y="17.78" rot="R180"/>
 <instance part="R9" gate="G$1" x="66.04" y="-10.16" rot="R180"/>
 <instance part="GND6" gate="1" x="55.88" y="-17.78"/>
+<instance part="R10" gate="G$1" x="73.66" y="27.94" rot="R270"/>
+<instance part="R11" gate="G$1" x="73.66" y="0" rot="R270"/>
+<instance part="R12" gate="G$1" x="203.2" y="30.48" rot="R270"/>
+<instance part="LED1" gate="G$1" x="203.2" y="17.78" rot="R180"/>
 </instances>
 <busses>
@@
 <pinref part="R8" gate="G$1" pin="2"/>
 <pinref part="GND6" gate="1" pin="GND"/>
-<wire x1="60.96" y1="10.16" x2="55.88" y2="10.16" width="0.1524" layer="91"/>
-<wire x1="55.88" y1="10.16" x2="55.88" y2="-10.16" width="0.1524" layer="91"/>
+<wire x1="60.96" y1="17.78" x2="55.88" y2="17.78" width="0.1524" layer="91"/>
+<wire x1="55.88" y1="17.78" x2="55.88" y2="-10.16" width="0.1524" layer="91"/>
 <pinref part="R9" gate="G$1" pin="2"/>
 <wire x1="55.88" y1="-10.16" x2="55.88" y2="-15.24" width="0.1524" layer="91"/>
 <wire x1="60.96" y1="-10.16" x2="55.88" y2="-10.16" width="0.1524" layer="91"/>
 <junction x="55.88" y="-10.16"/>
+</segment>
+<segment>
+<wire x1="203.2" y1="15.24" x2="203.2" y2="7.62" width="0.1524" layer="91"/>
+<label x="203.2" y="10.16" size="1.778" layer="95"/>
+<pinref part="LED1" gate="G$1" pin="A"/>
 </segment>
 </net>
@@
 </segment>
 <segment>
-<pinref part="BTN1" gate="G$1" pin="VCC"/>
-<wire x1="78.74" y1="15.24" x2="73.66" y2="15.24" width="0.1524" layer="91"/>
-<label x="71.12" y="15.24" size="1.778" layer="95"/>
-</segment>
-<segment>
-<pinref part="BTN2" gate="G$1" pin="VCC"/>
-<wire x1="78.74" y1="-5.08" x2="73.66" y2="-5.08" width="0.1524" layer="91"/>
-<label x="71.12" y="-5.08" size="1.778" layer="95"/>
+<wire x1="73.66" y1="33.02" x2="73.66" y2="38.1" width="0.1524" layer="91"/>
+<label x="73.66" y="38.1" size="1.778" layer="95"/>
+<pinref part="R10" gate="G$1" pin="1"/>
+</segment>
+<segment>
+<wire x1="73.66" y1="5.08" x2="73.66" y2="10.16" width="0.1524" layer="91"/>
+<label x="73.66" y="10.16" size="1.778" layer="95"/>
+<pinref part="R11" gate="G$1" pin="1"/>
 </segment>
 </net>
@@
 <pinref part="R8" gate="G$1" pin="1"/>
 <pinref part="BTN1" gate="G$1" pin="OUT"/>
-<wire x1="71.12" y1="10.16" x2="78.74" y2="10.16" width="0.1524" layer="91"/>
-<label x="71.374" y="7.366" size="1.778" layer="95"/>
+<wire x1="71.12" y1="17.78" x2="78.74" y2="17.78" width="0.1524" layer="91"/>
+<label x="71.374" y="14.986" size="1.778" layer="95"/>
 </segment>
 <segment>
@@
 </segment>
 </net>
+<net name="N$1" class="0">
+<segment>
+<pinref part="BTN1" gate="G$1" pin="VCC"/>
+<pinref part="R10" gate="G$1" pin="2"/>
+<wire x1="78.74" y1="22.86" x2="73.66" y2="22.86" width="0.1524" layer="91"/>
+</segment>
+</net>
+<net name="N$2" class="0">
+<segment>
+<pinref part="BTN2" gate="G$1" pin="VCC"/>
+<pinref part="R11" gate="G$1" pin="2"/>
+<wire x1="78.74" y1="-5.08" x2="73.66" y2="-5.08" width="0.1524" layer="91"/>
+</segment>
+</net>
+<net name="N$3" class="0">
+<segment>
+<pinref part="U1" gate="U$1" pin="PD5(T1)"/>
+<wire x1="203.2" y1="35.56" x2="175.26" y2="35.56" width="0.1524" layer="91"/>
+<pinref part="R12" gate="G$1" pin="1"/>
+</segment>
+</net>
+<net name="N$4" class="0">
+<segment>
+<pinref part="R12" gate="G$1" pin="2"/>
+<wire x1="203.2" y1="25.4" x2="203.2" y2="22.86" width="0.1524" layer="91"/>
+<pinref part="LED1" gate="G$1" pin="C"/>
+</segment>
+</net>

Commit message: Moved Button connectors away from screw keepout, fixed backwards LED1, rearranged SMD resistors around button connectors. No reported DRC/ERC errors
Connections:
- net GND: now also LED1.C; no longer LED1.A
- net N$4: now also LED1.A; no longer LED1.C
Other:
- moved on the sheet: LED1
Changed lines of the file:
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@@
 <?xml version="1.0" encoding="utf-8"?>
 <!DOCTYPE eagle SYSTEM "eagle.dtd">
-<eagle version="8.3.1">
+<eagle version="8.6.0">
 <drawing>
 <settings>
-<setting alwaysvectorfont="no"/>
+<setting alwaysvectorfont="yes"/>
 <setting verticaltext="up"/>
 </settings>
@@
 <layers>
 <layer number="1" name="Top" color="4" fill="1" visible="no" active="no"/>
+<layer number="2" name="Route2" color="1" fill="3" visible="no" active="no"/>
+<layer number="3" name="Route3" color="4" fill="3" visible="no" active="no"/>
+<layer number="4" name="Route4" color="1" fill="4" visible="no" active="no"/>
+<layer number="5" name="Route5" color="4" fill="4" visible="no" active="no"/>
+<layer number="6" name="Route6" color="1" fill="8" visible="no" active="no"/>
+<layer number="7" name="Route7" color="4" fill="8" visible="no" active="no"/>
+<layer number="8" name="Route8" color="1" fill="2" visible="no" active="no"/>
+<layer number="9" name="Route9" color="4" fill="2" visible="no" active="no"/>
+<layer number="10" name="Route10" color="1" fill="7" visible="no" active="no"/>
+<layer number="11" name="Route11" color="4" fill="7" visible="no" active="no"/>
+<layer number="12" name="Route12" color="1" fill="5" visible="no" active="no"/>
+<layer number="13" name="Route13" color="4" fill="5" visible="no" active="no"/>
+<layer number="14" name="Route14" color="1" fill="6" visible="no" active="no"/>
+<layer number="15" name="Route15" color="4" fill="6" visible="no" active="no"/>
 <layer number="16" name="Bottom" color="1" fill="1" visible="no" active="no"/>
 <layer number="17" name="Pads" color="2" fill="1" visible="no" active="no"/>
@@
 <layer number="59" name="tCarbon" color="7" fill="1" visible="no" active="no"/>
 <layer number="60" name="bCarbon" color="7" fill="1" visible="no" active="no"/>
+<layer number="88" name="SimResults" color="9" fill="1" visible="yes" active="yes"/>
+<layer number="89" name="SimProbes" color="9" fill="1" visible="yes" active="yes"/>
 <layer number="90" name="Modules" color="5" fill="1" visible="yes" active="yes"/>
 <layer number="91" name="Nets" color="2" fill="1" visible="yes" active="yes"/>
@@
 <instance part="R11" gate="G$1" x="73.66" y="0" rot="R270"/>
 <instance part="R12" gate="G$1" x="203.2" y="30.48" rot="R270"/>
-<instance part="LED1" gate="G$1" x="203.2" y="17.78" rot="R180"/>
+<instance part="LED1" gate="G$1" x="203.2" y="20.32"/>
 </instances>
 <busses>
@@
 <wire x1="203.2" y1="15.24" x2="203.2" y2="7.62" width="0.1524" layer="91"/>
 <label x="203.2" y="10.16" size="1.778" layer="95"/>
-<pinref part="LED1" gate="G$1" pin="A"/>
+<pinref part="LED1" gate="G$1" pin="C"/>
 </segment>
 </net>
@@
 <segment>
 <pinref part="R12" gate="G$1" pin="2"/>
+<pinref part="LED1" gate="G$1" pin="A"/>
 <wire x1="203.2" y1="25.4" x2="203.2" y2="22.86" width="0.1524" layer="91"/>
-<pinref part="LED1" gate="G$1" pin="C"/>
-</segment>
-</net>
+</segment>
+</net>
